File: Diseño placa/Diseño placa.sch (KiCad schematic (older format))
At the start: 23 parts

Commit message: Avances esquemático en Kicad
Parts:
- removed C? (x2): 4.7n, symbol C
- removed C?: 47n, symbol C
- removed IC?: ATMEGA32-A, TQFP44, symbol ATMEGA32-A
- removed R? (x3): 1k, symbol R
- removed R? (x3): 33k, symbol R
- removed R? (x3): 100k, symbol R
- removed R? (x2): 2.2k, symbol R
- removed R?: 20M, symbol R
- removed R?: 10k, symbol R
- removed R?: 150k, symbol R
- removed R?: 200k, symbol R
- removed U? (x4): LM741, symbol LM741
- added C1, C2: 10u, symbol C
- added C10, C20, C21, C9: 4.7n, symbol C
- added C11, C12, C15, C16, C17, C22, C24, C25, C26, C27, C3, C4, C5, C?: 100n, symbol C
- added C13, C19, C8: 47n, symbol C
- added C14: 1n, symbol C
- added C18, C23: 1u, symbol C
- added C6, C7: 10p, symbol C
- added IC?: ATMEGA32-P, DIL40, symbol ATMEGA32-P
- added M1: DIL24, symbol DIL24
- added R1, R11, R15, R18, R25: 10k, symbol R
- added R10, R12, R20, R4: 1k, symbol R
- added R13: 22k, symbol R
- added R14, R17, R26, R27, R9: 100k, symbol R
- added R16: 100, symbol R
- added R19: 1.2M, symbol R
- added R2: 3.3k, symbol R
- added R21, R22, R5, R6: 33k, symbol R
- added R23, R24, R7, R8: 2.2k, symbol R
- added R28: 330k, symbol R
- added R3: 470k, symbol R
- added Re: R, symbol R
- added SW1: SW_PUSH, symbol SW_PUSH
- added U1, U2, U3, U4, U5, U?: OPA625, symbol OPA625
- added U?: LM317AT, TO-220, symbol LM317AT
- added X1: 16M, symbol Crystal
Connections:
- net labels added: ADC_OFF, MUX16, OFFSET, RESET, VCC, VCC/2
- net labels removed: Vcc, vssop
- wire segments 44 -> 127
