File: Diseño placa/Diseño-placa.sch (KiCad schematic (older format))
At the start: 89 parts, among them IC1 ATMEGA32-P, M1 DIL24, M2 DIL24, M3 DIL16, P1 CONN_01X03, P2 CONN_02X08, P3 CONN_01X01, P4 CONN_01X16, P5 CONN_01X05, P6 CONN_01X05, P7 CONN_02X03, SW1 SW_PUSH, SW2 SW_PUSH, SW3 SW_PUSH, SW4 SW_PUSH, SW5 SW_PUSH, U1 REG104, U2 OPA625, U3 OPA625, U4 OPA625, U5 OPA625, U6 OPA625, U7 OPA625, X1 16M

Commit message: PCB corrección de pistas conflictivas
Parts:
- C10, C11, C12, C18, C19, C2, C20, C22, C23, C25, C26, C27, C29, C30, C31, C32, C4, C5, C6, C8, C9: footprint Capacitors_ThroughHole:C_Rect_L4_W2.5_P2.5 -> Capacitors_ThroughHole:C_Rect_L7_W6_P5
- C13, C14, C15, C16: footprint Capacitors_ThroughHole:C_Rect_L4_W2.5_P2.5 -> Capacitors_ThroughHole:C_Rect_L13_W4_P10
- C17, C24: footprint Capacitors_ThroughHole:C_Rect_L7_W6_P5 -> Capacitors_ThroughHole:C_Rect_L27_W11_P22
Changed lines of the file:
@@
 F 0 "C9" H 4775 1850 50  0000 L CNN
 F 1 "47n" H 4775 1650 50  0000 L CNN
-F 2 "Capacitors_ThroughHole:C_Rect_L4_W2.5_P2.5" H 4788 1600 30  0001 C CNN
+F 2 "Capacitors_ThroughHole:C_Rect_L7_W6_P5" H 4788 1600 30  0001 C CNN
 F 3 "" H 4750 1750 60  0000 C CNN
 	1    4750 1750
@@
 F 0 "C13" H 5925 1750 50  0000 L CNN
 F 1 "4.7n" H 5925 1550 50  0000 L CNN
-F 2 "Capacitors_ThroughHole:C_Rect_L4_W2.5_P2.5" H 5938 1500 30  0001 C CNN
+F 2 "Capacitors_ThroughHole:C_Rect_L13_W4_P10" H 5938 1500 30  0001 C CNN
 F 3 "" H 5900 1650 60  0000 C CNN
 	1    5900 1650
@@
 F 0 "C16" H 6125 850 50  0000 L CNN
 F 1 "4.7n" H 6125 650 50  0000 L CNN
-F 2 "Capacitors_ThroughHole:C_Rect_L4_W2.5_P2.5" H 6138 600 30  0001 C CNN
+F 2 "Capacitors_ThroughHole:C_Rect_L13_W4_P10" H 6138 600 30  0001 C CNN
 F 3 "" H 6100 750 60  0000 C CNN
 	1    6100 750
@@
 F 0 "C19" H 8875 2950 50  0000 L CNN
 F 1 "47n" H 8875 2750 50  0000 L CNN
-F 2 "Capacitors_ThroughHole:C_Rect_L4_W2.5_P2.5" H 8888 2700 30  0001 C CNN
+F 2 "Capacitors_ThroughHole:C_Rect_L7_W6_P5" H 8888 2700 30  0001 C CNN
 F 3 "" H 8850 2850 60  0000 C CNN
 	1    8850 2850
@@
 F 0 "C20" H 9625 3800 50  0000 L CNN
 F 1 "100n" H 9625 3600 50  0000 L CNN
-F 2 "Capacitors_ThroughHole:C_Rect_L4_W2.5_P2.5" H 9638 3550 30  0001 C CNN
+F 2 "Capacitors_ThroughHole:C_Rect_L7_W6_P5" H 9638 3550 30  0001 C CNN
 F 3 "" H 9600 3700 60  0000 C CNN
 	1    9600 3700
@@
 F 0 "C24" H 10575 4900 50  0000 L CNN
 F 1 "1u" H 10575 4700 50  0000 L CNN
-F 2 "Capacitors_ThroughHole:C_Rect_L7_W6_P5" H 10588 4650 30  0001 C CNN
+F 2 "Capacitors_ThroughHole:C_Rect_L27_W11_P22" H 10588 4650 30  0001 C CNN
 F 3 "" H 10550 4800 60  0000 C CNN
 	1    10550 4800
@@
 F 0 "C15" H 6075 3450 50  0000 L CNN
 F 1 "4.7n" H 6075 3250 50  0000 L CNN
-F 2 "Capacitors_ThroughHole:C_Rect_L4_W2.5_P2.5" H 6088 3200 30  0001 C CNN
+F 2 "Capacitors_ThroughHole:C_Rect_L13_W4_P10" H 6088 3200 30  0001 C CNN
 F 3 "" H 6050 3350 60  0000 C CNN
 	1    6050 3350
@@
 F 0 "C14" H 6075 2550 50  0000 L CNN
 F 1 "4.7n" H 6075 2350 50  0000 L CNN
-F 2 "Capacitors_ThroughHole:C_Rect_L4_W2.5_P2.5" H 6088 2300 30  0001 C CNN
+F 2 "Capacitors_ThroughHole:C_Rect_L13_W4_P10" H 6088 2300 30  0001 C CNN
 F 3 "" H 6050 2450 60  0000 C CNN
 	1    6050 2450
@@
 F 0 "C17" H 7825 3350 50  0000 L CNN
 F 1 "1u" H 7825 3150 50  0000 L CNN
-F 2 "Capacitors_ThroughHole:C_Rect_L7_W6_P5" H 7838 3100 30  0001 C CNN
+F 2 "Capacitors_ThroughHole:C_Rect_L27_W11_P22" H 7838 3100 30  0001 C CNN
 F 3 "" H 7800 3250 60  0000 C CNN
 	1    7800 3250
@@
 F 0 "C22" H 9975 6050 50  0000 L CNN
 F 1 "100n" H 9975 5850 50  0000 L CNN
-F 2 "Capacitors_ThroughHole:C_Rect_L4_W2.5_P2.5" H 9988 5800 30  0001 C CNN
+F 2 "Capacitors_ThroughHole:C_Rect_L7_W6_P5" H 9988 5800 30  0001 C CNN
 F 3 "" H 9950 5950 60  0000 C CNN
 	1    9950 5950
@@
 F 0 "C18" H 8125 6050 50  0000 L CNN
 F 1 "100n" H 8125 5850 50  0000 L CNN
-F 2 "Capacitors_ThroughHole:C_Rect_L4_W2.5_P2.5" H 8138 5800 30  0001 C CNN
+F 2 "Capacitors_ThroughHole:C_Rect_L7_W6_P5" H 8138 5800 30  0001 C CNN
 F 3 "" H 8100 5950 60  0000 C CNN
 	1    8100 5950
@@
 F 0 "C4" H 1375 3050 50  0000 L CNN
 F 1 "100n" H 1375 2850 50  0000 L CNN
-F 2 "Capacitors_ThroughHole:C_Rect_L4_W2.5_P2.5" H 1388 2800 30  0001 C CNN
+F 2 "Capacitors_ThroughHole:C_Rect_L7_W6_P5" H 1388 2800 30  0001 C CNN
 F 3 "" H 1350 2950 60  0000 C CNN
 	1    1350 2950
@@
 F 0 "C8" H 2925 1250 50  0000 L CNN
 F 1 "100n" H 2925 1050 50  0000 L CNN
-F 2 "Capacitors_ThroughHole:C_Rect_L4_W2.5_P2.5" H 2938 1000 30  0001 C CNN
+F 2 "Capacitors_ThroughHole:C_Rect_L7_W6_P5" H 2938 1000 30  0001 C CNN
 F 3 "" H 2900 1150 60  0000 C CNN
 	1    2900 1150
@@
 F 0 "C2" H 1325 6250 50  0000 L CNN
 F 1 "100n" H 1325 6050 50  0000 L CNN
-F 2 "Capacitors_ThroughHole:C_Rect_L4_W2.5_P2.5" H 1338 6000 30  0001 C CNN
+F 2 "Capacitors_ThroughHole:C_Rect_L7_W6_P5" H 1338 6000 30  0001 C CNN
 F 3 "" H 1300 6150 60  0000 C CNN
 	1    1300 6150
@@
 F 0 "C11" H 5225 1000 50  0000 L CNN
 F 1 "100n" H 5225 800 50  0000 L CNN
-F 2 "Capacitors_ThroughHole:C_Rect_L4_W2.5_P2.5" H 5238 750 30  0001 C CNN
+F 2 "Capacitors_ThroughHole:C_Rect_L7_W6_P5" H 5238 750 30  0001 C CNN
 F 3 "" H 5200 900 60  0000 C CNN
 	1    5200 900
@@
 F 0 "C10" H 4925 3550 50  0000 L CNN
 F 1 "47n" H 4925 3350 50  0000 L CNN
-F 2 "Capacitors_ThroughHole:C_Rect_L4_W2.5_P2.5" H 4938 3300 30  0001 C CNN
+F 2 "Capacitors_ThroughHole:C_Rect_L7_W6_P5" H 4938 3300 30  0001 C CNN
 F 3 "" H 4900 3450 60  0000 C CNN
 	1    4900 3450
@@
 F 0 "C5" H 1475 7150 50  0000 L CNN
 F 1 "100n" H 1475 6950 50  0000 L CNN
-F 2 "Capacitors_ThroughHole:C_Rect_L4_W2.5_P2.5" H 1488 6900 30  0001 C CNN
+F 2 "Capacitors_ThroughHole:C_Rect_L7_W6_P5" H 1488 6900 30  0001 C CNN
 F 3 "" H 1450 7050 60  0000 C CNN
 	1    1450 7050
@@
 F 0 "C6" H 2125 7450 50  0000 L CNN
 F 1 "10n" H 2125 7250 50  0000 L CNN
-F 2 "Capacitors_ThroughHole:C_Rect_L4_W2.5_P2.5" H 2138 7200 30  0001 C CNN
+F 2 "Capacitors_ThroughHole:C_Rect_L7_W6_P5" H 2138 7200 30  0001 C CNN
 F 3 "" H 2100 7350 60  0000 C CNN
 	1    2100 7350
@@
 F 0 "C25" H 10725 1100 50  0000 L CNN
 F 1 "100n" H 10725 900 50  0000 L CNN
-F 2 "Capacitors_ThroughHole:C_Rect_L4_W2.5_P2.5" H 10738 850 30  0001 C CNN
+F 2 "Capacitors_ThroughHole:C_Rect_L7_W6_P5" H 10738 850 30  0001 C CNN
 F 3 "" H 10700 1000 60  0000 C CNN
 	1    10700 1000
@@
 F 0 "C26" H 10775 2500 50  0000 L CNN
 F 1 "100n" H 10775 2300 50  0000 L CNN
-F 2 "Capacitors_ThroughHole:C_Rect_L4_W2.5_P2.5" H 10788 2250 30  0001 C CNN
+F 2 "Capacitors_ThroughHole:C_Rect_L7_W6_P5" H 10788 2250 30  0001 C CNN
 F 3 "" H 10750 2400 60  0000 C CNN
 	1    10750 2400
@@
 F 0 "C23" H 10475 4050 50  0000 L CNN
 F 1 "100n" H 10475 3850 50  0000 L CNN
-F 2 "Capacitors_ThroughHole:C_Rect_L4_W2.5_P2.5" H 10488 3800 30  0001 C CNN
+F 2 "Capacitors_ThroughHole:C_Rect_L7_W6_P5" H 10488 3800 30  0001 C CNN
 F 3 "" H 10450 3950 60  0000 C CNN
 	1    10450 3950
@@
 F 0 "C27" H 10875 5900 50  0000 L CNN
 F 1 "100n" H 10875 5700 50  0000 L CNN
-F 2 "Capacitors_ThroughHole:C_Rect_L4_W2.5_P2.5" H 10888 5650 30  0001 C CNN
+F 2 "Capacitors_ThroughHole:C_Rect_L7_W6_P5" H 10888 5650 30  0001 C CNN
 F 3 "" H 10850 5800 60  0000 C CNN
 	1    10850 5800
@@
 F 0 "C12" H 5225 2700 50  0000 L CNN
 F 1 "100n" H 5225 2500 50  0000 L CNN
-F 2 "Capacitors_ThroughHole:C_Rect_L4_W2.5_P2.5" H 5238 2450 30  0001 C CNN
+F 2 "Capacitors_ThroughHole:C_Rect_L7_W6_P5" H 5238 2450 30  0001 C CNN
 F 3 "" H 5200 2600 60  0000 C CNN
 	1    5200 2600
@@
 F 0 "C29" H 2775 5750 50  0000 L CNN
 F 1 "100n" H 2775 5550 50  0000 L CNN
-F 2 "Capacitors_ThroughHole:C_Rect_L4_W2.5_P2.5" H 2788 5500 30  0001 C CNN
+F 2 "Capacitors_ThroughHole:C_Rect_L7_W6_P5" H 2788 5500 30  0001 C CNN
 F 3 "" H 2750 5650 60  0000 C CNN
 	1    2750 5650
@@
 F 0 "C31" H 3825 5750 50  0000 L CNN
 F 1 "100n" H 3825 5550 50  0000 L CNN
-F 2 "Capacitors_ThroughHole:C_Rect_L4_W2.5_P2.5" H 3838 5500 30  0001 C CNN
+F 2 "Capacitors_ThroughHole:C_Rect_L7_W6_P5" H 3838 5500 30  0001 C CNN
 F 3 "" H 3800 5650 60  0000 C CNN
 	1    3800 5650
@@
 F 0 "C30" H 2775 6250 50  0000 L CNN
 F 1 "100n" H 2775 6050 50  0000 L CNN
-F 2 "Capacitors_ThroughHole:C_Rect_L4_W2.5_P2.5" H 2788 6000 30  0001 C CNN
+F 2 "Capacitors_ThroughHole:C_Rect_L7_W6_P5" H 2788 6000 30  0001 C CNN
 F 3 "" H 2750 6150 60  0000 C CNN
 	1    2750 6150
@@
 F 0 "C32" H 3875 6250 50  0000 L CNN
 F 1 "100n" H 3875 6050 50  0000 L CNN
-F 2 "Capacitors_ThroughHole:C_Rect_L4_W2.5_P2.5" H 3888 6000 30  0001 C CNN
+F 2 "Capacitors_ThroughHole:C_Rect_L7_W6_P5" H 3888 6000 30  0001 C CNN
 F 3 "" H 3850 6150 60  0000 C CNN
 	1    3850 6150

Commit message: Más informe
Parts:
- removed R2: 470k, Resistors_ThroughHole:Resistor_Horizontal_RM10mm, symbol R
Connections:
- net MUX2IO: now also C9.1, R4.1, R6.2
Changed lines of the file:
@@
 $EndDescr
-$Comp
-L R R2
-U 1 1 563C57F5
-P 4500 1350
-F 0 "R2" V 4580 1350 50  0000 C CNN
-F 1 "470k" V 4500 1350 50  0000 C CNN
-F 2 "Resistors_ThroughHole:Resistor_Horizontal_RM10mm" V 4430 1350 30  0001 C CNN
-F 3 "" H 4500 1350 30  0000 C CNN
-	1    4500 1350
-	0    1    1    0
-$EndComp
 $Comp
 L C C9
@@
 Text Label 4400 2050 0    60   ~ 0
 VCC/2
-Text Label 4000 1350 0    60   ~ 0
+Text Label 4300 1350 0    60   ~ 0
 MUX2IO
 Text Label 8650 5200 0    60   ~ 0
@@
 	4500 3050 4150 3050
 Wire Wire Line
-	4000 1350 4350 1350
+	4300 1350 4650 1350
 Wire Wire Line
 	1350 3250 1350 3100
